Commit message: rp_ rename package

File: rp_urdf_description/urdf/RobotPallet_urdf.xacro (robot description, xacro)
@@ -1,7 +1,7 @@
 <?xml version="1.0" ?>
-<robot name="RobotPallet_urdf" xmlns:xacro="http://www.ros.org/wiki/xacro">
-<xacro:include filename="$(find RobotPallet_urdf_description)/urdf/materials.xacro" />
-<xacro:include filename="$(find RobotPallet_urdf_description)/urdf/RobotPallet_urdf.trans" />
-<xacro:include filename="$(find RobotPallet_urdf_description)/urdf/RobotPallet_urdf_gazebo.xacro" />
+<robot name="rp_urdf" xmlns:xacro="http://www.ros.org/wiki/xacro">
+<xacro:include filename="$(find rp_urdf_description)/urdf/materials.xacro" />
+<xacro:include filename="$(find rp_urdf_description)/urdf/rp_urdf.trans" />
+<xacro:include filename="$(find rp_urdf_description)/urdf/rp_urdf_gazebo.xacro" />
 <link name="base_link">
   <inertial>
@@ -13,5 +13,5 @@
     <origin rpy="0 0 0" xyz="0 0 0"/>
     <geometry>
-      <mesh filename="package://RobotPallet_urdf_description/meshes/base_link.stl" scale="0.001 0.001 0.001"/>
+      <mesh filename="package://rp_urdf_description/meshes/base_link.stl" scale="0.001 0.001 0.001"/>
     </geometry>
     <material name="silver"/>
@@ -20,5 +20,5 @@
     <origin rpy="0 0 0" xyz="0 0 0"/>
     <geometry>
-      <mesh filename="package://RobotPallet_urdf_description/meshes/base_link.stl" scale="0.001 0.001 0.001"/>
+      <mesh filename="package://rp_urdf_description/meshes/base_link.stl" scale="0.001 0.001 0.001"/>
     </geometry>
   </collision>
@@ -33,5 +33,5 @@
     <origin rpy="0 0 0" xyz="-0.172949 -1.301919 -0.016779"/>
     <geometry>
-      <mesh filename="package://RobotPallet_urdf_description/meshes/caster_der_1.stl" scale="0.001 0.001 0.001"/>
+      <mesh filename="package://rp_urdf_description/meshes/caster_der_1.stl" scale="0.001 0.001 0.001"/>
     </geometry>
     <material name="silver"/>
@@ -40,5 +40,5 @@
     <origin rpy="0 0 0" xyz="-0.172949 -1.301919 -0.016779"/>
     <geometry>
-      <mesh filename="package://RobotPallet_urdf_description/meshes/caster_der_1.stl" scale="0.001 0.001 0.001"/>
+      <mesh filename="package://rp_urdf_description/meshes/caster_der_1.stl" scale="0.001 0.001 0.001"/>
     </geometry>
   </collision>
@@ -53,5 +53,5 @@
     <origin rpy="0 0 0" xyz="0.247051 -1.301919 -0.016779"/>
     <geometry>
-      <mesh filename="package://RobotPallet_urdf_description/meshes/caster_izq_1.stl" scale="0.001 0.001 0.001"/>
+      <mesh filename="package://rp_urdf_description/meshes/caster_izq_1.stl" scale="0.001 0.001 0.001"/>
     </geometry>
     <material name="silver"/>
@@ -60,5 +60,5 @@
     <origin rpy="0 0 0" xyz="0.247051 -1.301919 -0.016779"/>
     <geometry>
-      <mesh filename="package://RobotPallet_urdf_description/meshes/caster_izq_1.stl" scale="0.001 0.001 0.001"/>
+      <mesh filename="package://rp_urdf_description/meshes/caster_izq_1.stl" scale="0.001 0.001 0.001"/>
     </geometry>
   </collision>
@@ -73,5 +73,5 @@
     <origin rpy="0 0 0" xyz="-0.331949 -0.128419 -0.103779"/>
     <geometry>
-      <mesh filename="package://RobotPallet_urdf_description/meshes/rueda_der_1.stl" scale="0.001 0.001 0.001"/>
+      <mesh filename="package://rp_urdf_description/meshes/rueda_der_1.stl" scale="0.001 0.001 0.001"/>
     </geometry>
     <material name="silver"/>
@@ -80,5 +80,5 @@
     <origin rpy="0 0 0" xyz="-0.331949 -0.128419 -0.103779"/>
     <geometry>
-      <mesh filename="package://RobotPallet_urdf_description/meshes/rueda_der_1.stl" scale="0.001 0.001 0.001"/>
+      <mesh filename="package://rp_urdf_description/meshes/rueda_der_1.stl" scale="0.001 0.001 0.001"/>
     </geometry>
   </collision>
@@ -93,5 +93,5 @@
     <origin rpy="0 0 0" xyz="0.406051 -0.128419 -0.103779"/>
     <geometry>
-      <mesh filename="package://RobotPallet_urdf_description/meshes/rueda_izq_1.stl" scale="0.001 0.001 0.001"/>
+      <mesh filename="package://rp_urdf_description/meshes/rueda_izq_1.stl" scale="0.001 0.001 0.001"/>
     </geometry>
     <material name="silver"/>
@@ -100,5 +100,5 @@
     <origin rpy="0 0 0" xyz="0.406051 -0.128419 -0.103779"/>
     <geometry>
-      <mesh filename="package://RobotPallet_urdf_description/meshes/rueda_izq_1.stl" scale="0.001 0.001 0.001"/>
+      <mesh filename="package://rp_urdf_description/meshes/rueda_izq_1.stl" scale="0.001 0.001 0.001"/>
     </geometry>
   </collision>
@@ -113,5 +113,5 @@
     <origin rpy="0 0 0" xyz="-0.135898 -0.25514 -1.193698"/>
     <geometry>
-      <mesh filename="package://RobotPallet_urdf_description/meshes/horquilla_der_1.stl" scale="0.001 0.001 0.001"/>
+      <mesh filename="package://rp_urdf_description/meshes/horquilla_der_1.stl" scale="0.001 0.001 0.001"/>
     </geometry>
     <material name="silver"/>
@@ -120,5 +120,5 @@
     <origin rpy="0 0 0" xyz="-0.135898 -0.25514 -1.193698"/>
     <geometry>
-      <mesh filename="package://RobotPallet_urdf_description/meshes/horquilla_der_1.stl" scale="0.001 0.001 0.001"/>
+      <mesh filename="package://rp_urdf_description/meshes/horquilla_der_1.stl" scale="0.001 0.001 0.001"/>
     </geometry>
   </collision>
@@ -133,5 +133,5 @@
     <origin rpy="0 0 0" xyz="0.284102 -0.25514 -1.193698"/>
     <geometry>
-      <mesh filename="package://RobotPallet_urdf_description/meshes/horquilla_izq_1.stl" scale="0.001 0.001 0.001"/>
+      <mesh filename="package://rp_urdf_description/meshes/horquilla_izq_1.stl" scale="0.001 0.001 0.001"/>
     </geometry>
     <material name="silver"/>
@@ -140,5 +140,5 @@
     <origin rpy="0 0 0" xyz="0.284102 -0.25514 -1.193698"/>
     <geometry>
-      <mesh filename="package://RobotPallet_urdf_description/meshes/horquilla_izq_1.stl" scale="0.001 0.001 0.001"/>
+      <mesh filename="package://rp_urdf_description/meshes/horquilla_izq_1.stl" scale="0.001 0.001 0.001"/>
     </geometry>
   </collision>

File: rp_urdf_description/urdf/RobotPallet_urdf_gazebo.xacro (robot description, xacro)
@@ -1,4 +1,4 @@
 <?xml version="1.0" ?>
-<robot name="RobotPallet_urdf" xmlns:xacro="http://www.ros.org/wiki/xacro">
+<robot name="rp_urdf" xmlns:xacro="http://www.ros.org/wiki/xacro">
   <!-- Begin - Gazebo definition -->
   <gazebo reference="base">

File: rp_urdf_description/urdf/materials.xacro (robot description, xacro)
@@ -1,4 +1,4 @@
 <?xml version="1.0" ?>
-<robot name="RobotPallet_urdf" xmlns:xacro="http://www.ros.org/wiki/xacro" >
+<robot name="rp_urdf" xmlns:xacro="http://www.ros.org/wiki/xacro" >
 <material name="silver">
   <color rgba="0.700 0.700 0.700 1.000"/>
