Commit message: teleop move direction fix

File: rp_urdf_description/urdf/rp_urdf.xacro (robot description, xacro)
@@ -158,5 +158,5 @@
   <parent link="base_link"/>
   <child link="rueda_der_1"/>
-  <axis xyz="1.0 0.0 0.0"/>
+  <axis xyz="-1.0 0.0 0.0"/>
 </joint>
 <joint name="rueda_izq_base_link" type="continuous">

File: rp_urdf_description/urdf/rp_urdf_gazebo.xacro (robot description, xacro)
@@ -7,6 +7,6 @@
  <!-- Ruedas motrices plugin for gazebo -->
   <gazebo reference="rueda_der_1">
-    <mu1>0.5</mu1>
-    <mu2>0.5</mu2>
+    <mu1>0.9</mu1>
+    <mu2>0.9</mu2>
     <kp>500000.0</kp>
     <kd>10.0</kd>
@@ -17,6 +17,6 @@
   </gazebo>
   <gazebo reference="rueda_izq_1">
-    <mu1>0.5</mu1>
-    <mu2>0.5</mu2>
+    <mu1>0.9</mu1>
+    <mu2>0.9</mu2>
     <kp>500000.0</kp>
     <kd>10.0</kd>
@@ -29,6 +29,6 @@
  <!-- Ruedas caster plugin for gazebo -->
   <gazebo reference="caster_izq_1">
-    <mu1>0.5</mu1>
-    <mu2>0.5</mu2>
+    <mu1>0.2</mu1>
+    <mu2>0.2</mu2>
     <kp>500000.0</kp>
     <kd>10.0</kd>
@@ -39,6 +39,6 @@
   </gazebo>
   <gazebo reference="caster_der_1">
-    <mu1>0.5</mu1>
-    <mu2>0.5</mu2>
+    <mu1>0.2</mu1>
+    <mu2>0.2</mu2>
     <kp>500000.0</kp>
     <kd>10.0</kd>
@@ -52,11 +52,11 @@
     <plugin name="differential_drive_controller" filename="libgazebo_ros_diff_drive.so">
       <alwaysOn>true</alwaysOn>
-      <updateRate>50</updateRate>
+      <updateRate>10</updateRate>
       <leftJoint>rueda_izq_base_link</leftJoint>
       <rightJoint>rueda_der_base_link</rightJoint>
       <wheelSeparation>0.840</wheelSeparation>
       <wheelDiameter>0.230</wheelDiameter>
-      <wheelAcceleration>0.1</wheelAcceleration>
-      <wheelTorque>20</wheelTorque>
+      <wheelAcceleration>0.02</wheelAcceleration>
+      <wheelTorque>1000</wheelTorque>
       <commandTopic>cmd_vel</commandTopic>
       <odometryTopic>odom</odometryTopic>

Commit message: add laser scanner for urdf

File: rp_urdf_description/urdf/rp_urdf.xacro (robot description, xacro)
@@ -7,6 +7,8 @@
   <inertial>
     <origin rpy="0 0 0" xyz="0.0 0.3452934919578558 0.1391905292373332"/>
-    <mass value="13.404713841955479"/>
-    <inertia ixx="4.45282" ixy="-0.000196" ixz="0.000249" iyy="1.596267" iyz="0.566652" izz="5.300151"/>
+    <mass value="1.404713841955479"/>
+    <inertia ixx="2.2124416e-03" ixy="-1.2294101e-05" ixz="3.4938785e-05"
+               iyy="2.1193702e-03" iyz="-5.0120904e-06"
+               izz="2.0064271e-03"/>
   </inertial>
   <visual>

File: rp_urdf_description/urdf/rp_urdf_gazebo.xacro (robot description, xacro)
@@ -12,5 +12,5 @@
     <kd>10.0</kd>
     <minDepth>0.001</minDepth>
-    <maxVel>0.1</maxVel>
+    <maxVel>0.5</maxVel>
     <fdir1>1 0 0</fdir1>
     <material>Gazebo/FlatBlack</material>
@@ -22,5 +22,5 @@
     <kd>10.0</kd>
     <minDepth>0.001</minDepth>
-    <maxVel>0.1</maxVel>
+    <maxVel>0.5</maxVel>
     <fdir1>1 0 0</fdir1>
     <material>Gazebo/FlatBlack</material>
@@ -29,20 +29,20 @@
  <!-- Ruedas caster plugin for gazebo -->
   <gazebo reference="caster_izq_1">
-    <mu1>0.2</mu1>
-    <mu2>0.2</mu2>
+    <mu1>0.1</mu1>
+    <mu2>0.1</mu2>
     <kp>500000.0</kp>
     <kd>10.0</kd>
     <minDepth>0.001</minDepth>
-    <maxVel>0.1</maxVel>
+    <maxVel>0.5</maxVel>
     <fdir1>1 0 0</fdir1>
     <material>Gazebo/FlatBlack</material>
   </gazebo>
   <gazebo reference="caster_der_1">
-    <mu1>0.2</mu1>
-    <mu2>0.2</mu2>
+    <mu1>0.1</mu1>
+    <mu2>0.1</mu2>
     <kp>500000.0</kp>
     <kd>10.0</kd>
     <minDepth>0.001</minDepth>
-    <maxVel>0.1</maxVel>
+    <maxVel>0.5</maxVel>
     <fdir1>1 0 0</fdir1>
     <material>Gazebo/FlatBlack</material>
@@ -73,4 +73,20 @@
   <gazebo reference="front_camera_link">
     <material>Gazebo/Blue</material>
+  </gazebo>
+<!-- IMU representation -->
+<gazebo reference="imu_link">
+    <material>Gazebo/Yellow</material>
+  </gazebo>
+   <!-- LIDAR IZQ representation -->
+  <gazebo reference="lidar_izq_link">
+    <material>Gazebo/Red</material>
+  </gazebo>
+   <!-- LIDAR CENTRAL representation -->
+  <gazebo reference="lidar_cen_link">
+    <material>Gazebo/Red</material>
+  </gazebo>
+    <!-- LIDAR DER representation -->
+  <gazebo reference="lidar_der_link">
+    <material>Gazebo/Red</material>
   </gazebo>
  <gazebo reference="front_camera_link">
@@ -116,3 +132,61 @@
 </gazebo>
   <!-- End - Deep camera plugin -->
+  <!-- imu_link -->
+   <gazebo reference="imu_link">
+    <gravity>true</gravity>
+    <sensor name="imu_sensor" type="imu">
+      <always_on>true</always_on>
+      <update_rate>100</update_rate>
+      <visualize>true</visualize>
+      <topic>__default_topic__</topic>
+      <plugin filename="libgazebo_ros_imu_sensor.so" name="imu_plugin">
+        <topicName>imu</topicName>
+        <bodyName>imu_link</bodyName>
+        <updateRateHZ>10.0</updateRateHZ>
+        <gaussianNoise>0.0</gaussianNoise>
+        <xyzOffset>0 0 0</xyzOffset>
+        <rpyOffset>0 0 0</rpyOffset>
+        <frameName>imu_link</frameName>
+        <initialOrientationAsReference>false</initialOrientationAsReference>
+      </plugin>
+      <pose>0 0 0 0 0 0</pose>
+    </sensor>
+  </gazebo>
+  <!-- imu_link  end-->
+    <!-- laser2 -->
+  <gazebo reference="lidar_cen_link">
+    <sensor type="gpu_ray" name="head_hokuyo_sensor2">
+      <pose>0 0 0 0 0 0</pose>
+      <visualize>false</visualize>
+      <update_rate>40</update_rate>
+      <ray>
+        <scan>
+          <horizontal>
+            <samples>720</samples>
+            <resolution>1</resolution>
+            <min_angle>-1.570796</min_angle>
+            <max_angle>1.570796</max_angle>
+          </horizontal>
+        </scan>
+        <range>
+          <min>0.10</min>
+          <max>30.0</max>
+          <resolution>0.01</resolution>
+        </range>
+        <noise>
+          <type>gaussian</type>
+          <!-- Noise parameters based on published spec for Hokuyo laser
+               achieving "+-30mm" accuracy at range < 10m.  A mean of 0.0m and
+               stddev of 0.01m will put 99.7% of samples within 0.03m of the true
+               reading. -->
+          <mean>0.0</mean>
+          <stddev>0.01</stddev>
+        </noise>
+      </ray>
+      <plugin name="gazebo_ros_head_hokuyo_controller" filename="libgazebo_ros_gpu_laser.so">
+        <topicName>/rrbot/laser1/scan</topicName>
+        <frameName>lidar_cen_link</frameName>
+      </plugin>
+    </sensor>
+  </gazebo>
 </robot>
